Commit message: change sizes of Bubble man

File: models/bubbleperson.urdf (robot description, URDF)
Before this commit: robot bubble_man, 14 links, 13 joints
Links:
- link head: mass 5.0 -> 8.0; geometry collision sphere radius=0.24; visual sphere radius=0.24
- link left_foot: mass 2.0 -> 3.0; geometry collision sphere radius=0.12; visual sphere radius=0.12
- link left_hand: mass 1.0 -> 2.0; geometry collision sphere radius=0.10; visual sphere radius=0.10
- link left_lower_arm: mass 2.0 -> 3.0; geometry collision sphere radius=0.12; visual sphere radius=0.12
- link left_lower_leg: mass 5.0 -> 8.0; geometry collision sphere radius=0.16; visual sphere radius=0.16
- link left_upper_arm: mass 3.0 -> 5.0; geometry collision sphere radius=0.16; visual sphere radius=0.16
- link left_upper_leg: mass 8.0 -> 12.0; geometry collision sphere radius=0.20; visual sphere radius=0.20
- link right_foot: mass 2.0 -> 3.0; geometry collision sphere radius=0.12; visual sphere radius=0.12
- link right_hand: mass 1.0 -> 2.0; geometry collision sphere radius=0.10; visual sphere radius=0.10
- link right_lower_arm: mass 2.0 -> 3.0; geometry collision sphere radius=0.12; visual sphere radius=0.12
- link right_lower_leg: mass 5.0 -> 8.0; geometry collision sphere radius=0.16; visual sphere radius=0.16
- link right_upper_arm: mass 3.0 -> 5.0; geometry collision sphere radius=0.16; visual sphere radius=0.16
- link right_upper_leg: mass 8.0 -> 12.0; geometry collision sphere radius=0.20; visual sphere radius=0.20
- link torso: mass 20.0 -> 35.0; geometry collision sphere radius=0.50; visual sphere radius=0.50
Joints:
- joint left_ankle: origin xyz=0 0 -0.2 rpy=0 0 0 -> xyz=0 0 -0.4 rpy=0 0 0
- joint left_elbow: origin xyz=-0.2 0 0 rpy=0 0 0 -> xyz=-0.4 0 0 rpy=0 0 0
- joint left_hip: origin xyz=-0.12 0 -0.3 rpy=0 0 0 -> xyz=-0.24 0 -0.6 rpy=0 0 0
- joint left_knee: origin xyz=0 0 -0.25 rpy=0 0 0 -> xyz=0 0 -0.50 rpy=0 0 0
- joint left_shoulder: origin xyz=-0.3 0 0.1 rpy=0 0 0 -> xyz=-0.6 0 0.2 rpy=0 0 0
- joint left_wrist: origin xyz=-0.15 0 0 rpy=0 0 0 -> xyz=-0.30 0 0 rpy=0 0 0
- joint neck: origin xyz=0 0 0.3 rpy=0 0 0 -> xyz=0 0 0.6 rpy=0 0 0
- joint right_ankle: origin xyz=0 0 -0.2 rpy=0 0 0 -> xyz=0 0 -0.4 rpy=0 0 0
- joint right_elbow: origin xyz=0.2 0 0 rpy=0 0 0 -> xyz=0.4 0 0 rpy=0 0 0
- joint right_hip: origin xyz=0.12 0 -0.3 rpy=0 0 0 -> xyz=0.24 0 -0.6 rpy=0 0 0
- joint right_knee: origin xyz=0 0 -0.25 rpy=0 0 0 -> xyz=0 0 -0.50 rpy=0 0 0
- joint right_shoulder: origin xyz=0.3 0 0.1 rpy=0 0 0 -> xyz=0.6 0 0.2 rpy=0 0 0
- joint right_wrist: origin xyz=0.15 0 0 rpy=0 0 0 -> xyz=0.30 0 0 rpy=0 0 0
